File: KiCad/PlusD_Clone_MOD_1_2.kicad_pcb (KiCad board)
At the start: 2 copper layers, 98.6 x 99.1 mm, 65 parts, among them IC10 74LS27, IC12 L7805, IC5 74LS06, IC6 74LS126, IC9 74LS00, J1 ZX_CONNECTOR_GENERIC_SORTED, J2 FDD_CONNECTOR, J3 PARALLEL_CONNECTOR, J4 KEMPSTON, SW1 RESET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

Commit message: Add files via upload
Connections:
- net /SELROM3 renamed Net-(D3-Pad2)
- net /SELROM48 renamed Net-(D2-Pad2)
- net 9V renamed +9V
- C10 pad 2: 5V -> +5V
- C11 pad 2: 5V -> +5V
- C12 pad 2: 5V -> +5V
- C18 pad 1: 5V -> +5V
- C2 pad 2: 5V -> +5V
- C3 pad 2: 5V -> +5V
- C4 pad 2: 5V -> +5V
- C5 pad 2: 5V -> +5V
- C6 pad 2: 5V -> +5V
- C7 pad 2: 5V -> +5V
- C8 pad 2: 5V -> +5V
- C9 pad 2: 5V -> +5V
- IC10 pad 14: 5V -> +5V
- IC5 pad 14: 5V -> +5V
- IC6 pad 1: 5V -> +5V
- IC6 pad 10: 5V -> +5V
- IC6 pad 13: 5V -> +5V
- IC6 pad 14: 5V -> +5V
- IC9 pad 14: 5V -> +5V
- J4 pad 7: 5V -> +5V
- JP1 pad 2: 5V -> +5V
- R10 pad 2: 5V -> +5V
- R11 pad 2: 5V -> +5V
- R12 pad 2: 5V -> +5V
- R5 pad 2: 5V -> +5V
- U1 pad 15: 5V -> +5V
- U11 pad 24: 5V -> +5V
- U2 pad 28: 5V -> +5V
- U3 pad 28: 5V -> +5V
- U4 pad 24: 5V -> +5V
- U7 pad 20: 5V -> +5V
- U8 pad 16: 5V -> +5V
Routing:
- net +5V: track 0.00 -> 356.3 mm, vias 0 -> 1
- net 5V: track 402.8 -> 116.9 mm, vias 1 -> 3
- net A10: track 97.8 -> 151.8 mm, vias 2 -> 3
- net RD: track 182.8 -> 134.6 mm, vias 2 -> 4
- net A4: track 150.8 -> 187.0 mm, vias 1 -> 5
- net A0: track 93.7 -> 123.4 mm
- net Net-(IC5-Pad9): track 70.5 -> 99.9 mm
- net D1: track 170.0 -> 193.5 mm, vias 3 -> 4
- net RESET: track 133.6 -> 110.8 mm
- net Net-(IC9-Pad4): track 91.8 -> 114.4 mm, vias 2 -> 1
- net Net-(D1-Pad1): track 213.3 -> 190.9 mm, vias 3 -> 5
- net Net-(IC6-Pad9): track 56.6 -> 78.4 mm, vias 0 -> 1
- net A12: track 133.1 -> 112.2 mm, vias 1 -> 3
- net GND: track 591.0 -> 570.9 mm, vias 5 -> 0
- net Net-(C13-Pad2): track 134.7 -> 114.8 mm
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
Commit message: Add files via upload
Parts:
- moved SW3 2.59 mm to (65.5, 74.4)
Connections:
- JP6 pad 3: 5V -> +5V
- R1 pad 1: 5V -> +5V
- R2 pad 1: 5V -> +5V
- R3 pad 1: 5V -> +5V
- R4 pad 1: 5V -> +5V
- R6 pad 2: 5V -> +5V
- U3 pad 26: 5V -> +5V
Routing:
- net 5V: track 116.9 -> 0.00 mm, vias 3 -> 0
- net RD: track 134.6 -> 191.0 mm, vias 4 -> 2
- net Net-(IC9-Pad4): track 114.4 -> 76.3 mm, vias 1 -> 0
- net /MOTOR_ON: track 106.0 -> 68.0 mm, vias 0 -> 1
- net A10: track 151.8 -> 120.2 mm
- net A0: track 123.4 -> 92.2 mm, vias 2 -> 1
- net Net-(C13-Pad1): track 87.9 -> 59.5 mm, vias 0 -> 1
- net Net-(IC6-Pad9): track 78.4 -> 50.1 mm, vias 1 -> 0
- net D5: track 152.6 -> 179.5 mm, vias 1 -> 3
- net D7: track 195.7 -> 169.8 mm, vias 1 -> 2
- net A11: track 110.3 -> 84.9 mm, vias 2 -> 1
- net A14: track 69.1 -> 48.1 mm, vias 1 -> 2
- net D1: track 193.5 -> 172.4 mm, vias 4 -> 1
- net Net-(IC5-Pad9): track 99.9 -> 79.1 mm, vias 1 -> 2
- net Net-(C13-Pad2): track 114.8 -> 133.2 mm
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
Commit message: Add files via upload
Parts:
- SW4: footprint Button_Switch_THT:SW_ON_ON_SPDT_TH -> Button_Switch_THT:SW_CuK_OS102011MA1QN1_SPDT_Angled
- U2: value 27E257 -> W27E257
- moved SW2 16.0 mm to (94.0, 80.0)
- moved SW1 15.5 mm to (78.0, 80.0)
- moved SW3 1.55 mm to (65.8, 72.9)
- moved SW4 1.30 mm to (159.3, 93.7)
- moved JP1 1.08 mm to (90.9, 115.3)
- moved U3 0.27 mm to (126.5, 84.0)
- moved U2 0.26 mm to (126.5, 65.0)
- moved SW5 0.18 mm to (157.6, 34.4)
Routing:
- net D7: track 169.8 -> 229.8 mm, vias 2 -> 4
- net D4: track 171.1 -> 202.7 mm, vias 3 -> 1
- net Net-(IC12-Pad3): track 15.7 -> 40.5 mm
- net Net-(IC5-Pad9): track 79.1 -> 55.5 mm, vias 2 -> 1
- net D0: track 171.6 -> 194.1 mm
- net Net-(D1-Pad2): track 55.5 -> 77.9 mm
- net +5V: track 363.0 -> 384.9 mm
- net A3: track 164.0 -> 185.2 mm, vias 0 -> 1
- net /WDDIRC: track 55.9 -> 35.0 mm, vias 1 -> 0
- net A14: track 48.1 -> 66.3 mm, vias 2 -> 0
- net Net-(C13-Pad1): track 59.5 -> 77.5 mm, vias 1 -> 2
- net A7: track 80.4 -> 98.1 mm
- net A0: track 92.2 -> 109.4 mm, vias 1 -> 2
- net Net-(D1-Pad1): track 195.8 -> 212.8 mm, vias 1 -> 3
- net A4: track 175.4 -> 158.4 mm, vias 2 -> 3
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Other:
- board text added: "PCB MOD 1.2 by MerlinKV July 27, 2020"
- board text removed: "PCB MOD 1.2 by MerlinKV July 6, 2020"

Commit message: Add files via upload
Parts:
- U4: value PAL20L8 -> GAL20V8B
Other:
- board text added: "Original design by @Pachuquin & @alvaroalea"
- board text removed: "Original design by @alvaroalea"
Changed lines of the file:
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@@
       (effects (font (size 1 1) (thickness 0.15)))
     )
-    (fp_text value PAL20L8 (at 3.81 22.352) (layer F.SilkS)
+    (fp_text value GAL20V8B (at 3.81 22.352) (layer F.SilkS)
       (effects (font (size 1 1) (thickness 0.15)))
     )
@@
   (gr_line (start 86.868 114.3) (end 86.868 124.46) (layer Edge.Cuts) (width 0.15))
   (gr_line (start 63.5 114.3) (end 86.868 114.3) (layer Edge.Cuts) (width 0.15))
-  (gr_text "Original design by @alvaroalea" (at 91.694 98.806) (layer B.SilkS)
+  (gr_text "Original design by\n@Pachuquin & @alvaroalea" (at 80.01 99.187) (layer B.SilkS)
     (effects (font (size 1.5 1.5) (thickness 0.2)) (justify mirror))
   )
