File: KiCad/PlusD_Clone_MOD_1_2.sch (KiCad schematic (older format))
At the start: 61 parts, among them IC10 74LS27, IC12 L7805, IC5 74LS06, IC6 74LS126, IC9 74LS00, J1 ZX_CONNECTOR_GENERIC_SORTED, J2 FDD_CONNECTOR, J3 PARALLEL_CONNECTOR, J4 KEMPSTON, SW1 RESET, SW2 NMI, SW3 ROMSEL_JOY, SW4 ZX_SEL, SW5 ABBA, U1 WD1772, U11 GAL22V10, U2 27E257, U3 6264, U4 PAL20L8, U7 74LS374, U8 74LS175, Y1 8.000Mhz

Commit message: Add files via upload
Connections:
- net 5V: no longer C10.2, C11.2, C12.2, C18.1, C2.2, C3.2, C4.2, C5.2, C6.2, C7.2, C8.2, C9.2, IC10.14 (VCC), IC5.14 (VCC), IC6.1, IC6.10, IC6.13, IC6.14 (VCC), IC9.14 (VCC), J4.7, JP1.2 (Pin_2), R10.2, R11.2, R12.2, R5.2, U1.15 (VCC), U11.24 (VCC), U2.28 (VCC), U3.28 (VCC), U4.24 (VCC), U7.20 (VCC), U8.16 (VCC)
- net 9V renamed +9V
- net SELROM3: no longer names the net of D3.2 (A), D4.2 (A), SW4.1 (A)
- net SELROM48: no longer names the net of D2.2 (A), SW4.3 (C)
- new net +5V: C10.2, C11.2, C12.2, C18.1, C2.2, C3.2, C4.2, C5.2, C6.2, C7.2, C8.2, C9.2, IC10.14 (VCC), IC5.14 (VCC), IC6.1, IC6.10, IC6.13, IC6.14 (VCC), IC9.14 (VCC), J4.7, JP1.2 (Pin_2), R10.2, R11.2, R12.2, R5.2, U1.15 (VCC), U11.24 (VCC), U2.28 (VCC), U3.28 (VCC), U4.24 (VCC), U7.20 (VCC), U8.16 (VCC)
Other:
- moved on the sheet: R11, R12

Commit message: Add files via upload
Connections:
- net 5V is gone; now on net +5V: JP6.3 (B), R1.1, R2.1, R3.1, R4.1, R6.2, U3.26 (CE2)
Changed lines of the file:
@@
 U 5 1 5B5F7599
 P 10100 10350
-F 0 "IC6" H 9850 10700 50  0000 L CNN
+F 0 "IC6" H 9850 10700 39  0000 L CNN
 F 1 "74LS126" H 9950 10350 50  0000 L CNN
 F 2 "Package_DIP:DIP-14_W7.62mm_Socket_LongPads" H 10100 10350 50  0001 C CNN
@@
 U 5 1 5B5F76E6
 P 9600 10350
-F 0 "IC9" H 9850 10700 50  0000 R CNN
+F 0 "IC9" H 9850 10700 39  0000 R CNN
 F 1 "74LS00" H 9750 10350 50  0000 R CNN
 F 2 "Package_DIP:DIP-14_W7.62mm_Socket_LongPads" H 9600 10350 50  0001 C CNN
@@
 U 7 1 5B5F7893
 P 9100 10350
-F 0 "IC5" H 8950 10700 50  0000 C CNN
+F 0 "IC5" H 8950 10700 39  0000 C CNN
 F 1 "74LS06" H 9100 10350 50  0000 C CNN
 F 2 "Package_DIP:DIP-14_W7.62mm_Socket_LongPads" H 9100 10350 50  0001 C CNN
@@
 P 9050 8150
 F 0 "#PWR025" H 9050 7900 50  0001 C CNN
-F 1 "GND" H 9055 7977 50  0000 C CNN
+F 1 "GND" H 9055 7977 39  0000 C CNN
 F 2 "" H 9050 8150 50  0001 C CNN
 F 3 "" H 9050 8150 50  0001 C CNN
@@
 U 1 1 5B5C13B9
 P 10100 8300
-F 0 "R5" H 10030 8254 50  0000 R CNN
-F 1 "2K2" H 10030 8345 50  0000 R CNN
+F 0 "R5" H 10030 8254 39  0000 R CNN
+F 1 "2K2" H 10030 8345 39  0000 R CNN
 F 2 "Resistor_THT:R_Axial_DIN0207_L6.3mm_D2.5mm_P7.62mm_Horizontal" V 10030 8300 50  0001 C CNN
 F 3 "~" H 10100 8300 50  0001 C CNN
@@
 	-1   0    0    1
 $EndComp
-Text Label 6750 6000 0    50   ~ 0
-RESET
 $Comp
 L power:GND #PWR08
@@
 U 1 1 5C0B42C8
 P 2250 8200
-F 0 "R9" V 2450 8250 50  0000 R CNN
-F 1 "270" V 2350 8250 50  0000 R CNN
+F 0 "R9" V 2450 8250 39  0000 R CNN
+F 1 "270" V 2350 8250 39  0000 R CNN
 F 2 "Resistor_THT:R_Axial_DIN0207_L6.3mm_D2.5mm_P7.62mm_Horizontal" V 2180 8200 50  0001 C CNN
 F 3 "~" H 2250 8200 50  0001 C CNN
@@
 U 2 1 5C10F84E
 P 2800 8200
-F 0 "IC10" H 2800 8525 50  0000 C CNN
-F 1 "74LS27" H 2800 8434 50  0000 C CNN
+F 0 "IC10" H 2800 8525 39  0000 C CNN
+F 1 "74LS27" H 2800 8434 39  0000 C CNN
 F 2 "Package_DIP:DIP-14_W7.62mm_Socket_LongPads" H 2800 8200 50  0001 C CNN
 F 3 "" H 2800 8200 50  0001 C CNN
@@
 U 4 1 5C13DCAC
 P 3550 8500
-F 0 "IC9" H 3550 8183 50  0000 C CNN
-F 1 "74LS00" H 3550 8274 50  0000 C CNN
+F 0 "IC9" H 3550 8183 39  0000 C CNN
+F 1 "74LS00" H 3550 8274 39  0000 C CNN
 F 2 "Package_DIP:DIP-14_W7.62mm_Socket_LongPads" H 3550 8500 50  0001 C CNN
 F 3 "" H 3550 8500 50  0001 C CNN
@@
 U 4 1 5C13DF1E
 P 10600 10350
-F 0 "IC10" H 10850 10700 50  0000 R CNN
+F 0 "IC10" H 10850 10700 39  0000 R CNN
 F 1 "74LS27" H 10750 10350 50  0000 R CNN
 F 2 "Package_DIP:DIP-14_W7.62mm_Socket_LongPads" H 10600 10350 50  0001 C CNN
@@
 U 1 1 5C16DA38
 P 4500 8400
-F 0 "IC10" H 4500 8725 50  0000 C CNN
-F 1 "74LS27" H 4500 8634 50  0000 C CNN
+F 0 "IC10" H 4500 8725 39  0000 C CNN
+F 1 "74LS27" H 4500 8634 39  0000 C CNN
 F 2 "Package_DIP:DIP-14_W7.62mm_Socket_LongPads" H 4500 8400 50  0001 C CNN
 F 3 "" H 4500 8400 50  0001 C CNN
@@
 U 3 1 5C16DB22
 P 4500 8950
-F 0 "IC10" H 4500 9275 50  0000 C CNN
-F 1 "74LS27" H 4500 9184 50  0000 C CNN
+F 0 "IC10" H 4500 9275 39  0000 C CNN
+F 1 "74LS27" H 4500 9184 39  0000 C CNN
 F 2 "Package_DIP:DIP-14_W7.62mm_Socket_LongPads" H 4500 8950 50  0001 C CNN
 F 3 "" H 4500 8950 50  0001 C CNN
@@
 P 1900 8700
 F 0 "#PWR02" H 1900 8450 50  0001 C CNN
-F 1 "GND" H 1905 8527 50  0000 C CNN
+F 1 "GND" H 1905 8527 39  0000 C CNN
 F 2 "" H 1900 8700 50  0001 C CNN
 F 3 "" H 1900 8700 50  0001 C CNN
@@
 P 7925 9350
 F 0 "#PWR021" H 7925 9100 50  0001 C CNN
-F 1 "GND" H 7930 9177 50  0000 C CNN
+F 1 "GND" H 7930 9177 39  0000 C CNN
 F 2 "" H 7925 9350 50  0001 C CNN
 F 3 "" H 7925 9350 50  0001 C CNN
@@
 P 1250 4300
 F 0 "#PWR0101" H 1250 4050 50  0001 C CNN
-F 1 "GND" H 1255 4127 50  0000 C CNN
+F 1 "GND" H 1255 4127 39  0000 C CNN
 F 2 "" H 1250 4300 50  0001 C CNN
 F 3 "" H 1250 4300 50  0001 C CNN
@@
 Wire Wire Line
 	8100 1150 8200 1150
-Text GLabel 8100 950  1    39   Input ~ 0
-5V
 Text GLabel 2200 5200 2    39   Input ~ 0
 FDC_CS
@@
 Text GLabel 4950 4850 2    39   Input ~ 0
 D7
-Text GLabel 4950 5200 2    39   Input ~ 0
-5V
 Text GLabel 4950 5300 2    39   Input ~ 0
 RD
@@
 Wire Wire Line
 	3650 6700 3650 6500
-Text GLabel 3650 6500 1    39   Input ~ 0
-5V
-Text GLabel 8700 800  1    39   Input ~ 0
-5V
 Wire Wire Line
 	8700 950  8700 800
@@
 P 13500 7350
 F 0 "#PWR0109" H 13500 7100 50  0001 C CNN
-F 1 "GND" H 13505 7177 50  0000 C CNN
+F 1 "GND" H 13505 7177 39  0000 C CNN
 F 2 "" H 13500 7350 50  0001 C CNN
 F 3 "" H 13500 7350 50  0001 C CNN
@@
 Wire Wire Line
 	10150 4400 11050 4400
-Text Label 11700 3250 1    39   ~ 0
+Text Label 11700 3250 1    39   ~ 8
 DS0
 Wire Wire Line
@@
 Wire Wire Line
 	11400 1500 12050 1500
-Text Label 12800 2550 0    39   ~ 0
+Text Label 12800 2550 0    39   ~ 8
 GATE_WRITE
-Text Label 12800 2950 0    39   ~ 0
+Text Label 12800 2950 0    39   ~ 8
 HEAD
-Text Label 12800 2850 0    39   ~ 0
+Text Label 12800 2850 0    39   ~ 8
 DATA_READ
-Text Label 12800 2750 0    39   ~ 0
+Text Label 12800 2750 0    39   ~ 8
 WRITE_PROT
-Text Label 12800 2650 0    39   ~ 0
+Text Label 12800 2650 0    39   ~ 8
 TRACK_0
-Text Label 12800 2450 0    39   ~ 0
+Text Label 12800 2450 0    39   ~ 8
 DATA_WRITE
-Text Label 12800 2350 0    39   ~ 0
+Text Label 12800 2350 0    39   ~ 8
 STEP
-Text Label 12800 2250 0    39   ~ 0
+Text Label 12800 2250 0    39   ~ 8
 DIR
-Text Label 12800 2150 0    39   ~ 0
+Text Label 12800 2150 0    39   ~ 8
 MOTOR_ON
-Text Label 12800 1950 0    39   ~ 0
+Text Label 12800 1950 0    39   ~ 8
 DS1
-Text Label 12800 1750 0    39   ~ 0
+Text Label 12800 1750 0    39   ~ 8
 INDEX
 Wire Wire Line
@@
 Wire Wire Line
 	11800 1400 12050 1400
-Text Label 11950 3250 1    39   ~ 0
+Text Label 11950 3250 1    39   ~ 8
 DS1
 NoConn ~ 3750 2850
@@
 	-1   0    0    1
 $EndComp
-Text Label 7400 2750 0    39   ~ 0
+Text Label 7400 2750 0    39   ~ 8
 WDMOTOR
-Text Label 7400 2650 0    39   ~ 0
+Text Label 7400 2650 0    39   ~ 8
 WDDIRC
-Text Label 7400 2550 0    39   ~ 0
+Text Label 7400 2550 0    39   ~ 8
 WDSTEP
-Text Label 7400 2450 0    39   ~ 0
+Text Label 7400 2450 0    39   ~ 8
 WDWG
-Text Label 7400 2350 0    39   ~ 0
+Text Label 7400 2350 0    39   ~ 8
 WDWD
-Text Label 12450 7050 0    39   ~ 0
+Text Label 12450 7050 0    39   ~ 8
 P21
-Text Label 12450 6850 0    39   ~ 0
+Text Label 12450 6850 0    39   ~ 8
 P17
-Text Label 12450 6750 0    39   ~ 0
+Text Label 12450 6750 0    39   ~ 8
 P15
-Text Label 12450 6650 0    39   ~ 0
+Text Label 12450 6650 0    39   ~ 8
 P13
-Text Label 12450 6550 0    39   ~ 0
+Text Label 12450 6550 0    39   ~ 8
 P11
-Text Label 12450 6450 0    39   ~ 0
+Text Label 12450 6450 0    39   ~ 8
 P9
-Text Label 12450 6350 0    39   ~ 0
+Text Label 12450 6350 0    39   ~ 8
 P7
-Text Label 12450 6250 0    39   ~ 0
+Text Label 12450 6250 0    39   ~ 8
 P5
-Text Label 12450 6150 0    39   ~ 0
+Text Label 12450 6150 0    39   ~ 8
 P3
-Text Label 12450 6050 0    39   ~ 0
+Text Label 12450 6050 0    39   ~ 8
 P1
 Wire Wire Line
@@
 P 1400 10000
 F 0 "#PWR0114" H 1400 9850 50  0001 C CNN
-F 1 "+5V" H 1415 10173 50  0000 C CNN
+F 1 "+5V" H 1415 10165 39  0000 C CNN
 F 2 "" H 1400 10000 50  0001 C CNN
 F 3 "" H 1400 10000 50  0001 C CNN
@@
 	0    1    1    0
 $EndComp
+$Comp
+L power:+5V #PWR0128
+U 1 1 60EDA996
+P 5150 5200
+F 0 "#PWR0128" H 5150 5050 50  0001 C CNN
+F 1 "+5V" V 5165 5328 39  0000 L CNN
+F 2 "" H 5150 5200 50  0001 C CNN
+F 3 "" H 5150 5200 50  0001 C CNN
+	1    5150 5200
+	0    1    1    0
+$EndComp
+Wire Wire Line
+	4950 5200 5150 5200
+$Comp
+L power:+5V #PWR0129
+U 1 1 60F16BB6
+P 3650 6500
+F 0 "#PWR0129" H 3650 6350 50  0001 C CNN
+F 1 "+5V" H 3665 6665 39  0000 C CNN
+F 2 "" H 3650 6500 50  0001 C CNN
+F 3 "" H 3650 6500 50  0001 C CNN
+	1    3650 6500
+	1    0    0    -1
+$EndComp
+$Comp
+L power:+5V #PWR0130
+U 1 1 60F1997B
+P 8700 800
+F 0 "#PWR0130" H 8700 650 50  0001 C CNN
+F 1 "+5V" H 8715 965 39  0000 C CNN
+F 2 "" H 8700 800 50  0001 C CNN
+F 3 "" H 8700 800 50  0001 C CNN
+	1    8700 800
+	1    0    0    -1
+$EndComp
+$Comp
+L power:+5V #PWR0131
+U 1 1 60F19C6D
+P 8100 950
+F 0 "#PWR0131" H 8100 800 50  0001 C CNN
+F 1 "+5V" H 8115 1115 39  0000 C CNN
+F 2 "" H 8100 950 50  0001 C CNN
+F 3 "" H 8100 950 50  0001 C CNN
+	1    8100 950
+	1    0    0    -1
+$EndComp
 $EndSCHEMATC

Commit message: Add files via upload
Other:
- moved on the sheet: U2

Commit message: Add files via upload
Parts:
- SW4: footprint Button_Switch_THT:SW_ON_ON_SPDT_TH -> Button_Switch_THT:SW_CuK_OS102011MA1QN1_SPDT_Angled
- U2: value 27E257 -> W27E257
Other:
- note removed: "Pos 1 (2-1 5-4) - DS0 es DS0 y DS1 es DS1\nPos 2 (2-3 5-6) - DS0 es DS1 DS1 es DS0"
- moved on the sheet: U8

Commit message: Add files via upload
Parts:
- U4: value PAL20L8 -> GAL20V8B
Changed lines of the file:
@@
 P 1700 5000
 F 0 "U4" H 1675 5043 39  0000 C CNN
-F 1 "PAL20L8" H 1675 4968 39  0000 C CNN
+F 1 "GAL20V8B" H 1675 4968 39  0000 C CNN
 F 2 "Package_DIP:DIP-24_W7.62mm_Socket_LongPads" H 1700 5000 39  0001 C CNN
 F 3 "" H 1700 5000 39  0001 C CNN
