File: KiCad/PlusD_Clone_1_3.kicad_pcb (KiCad board)
At the start: 2 copper layers, 98.6 x 99.1 mm, 61 parts, among them IC10 74LS27, IC5 74LS06, IC6 74LS126, IC9 74LS00, J1 ZX_CONNECTOR_GENERIC_SORTED, J2 FDD_CONNECTOR, J3 PARALLEL_CONNECTOR, J4 KEMPSTON, SW1 RESET, SW2 NMI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

Commit message: Add files via upload
Other:
- board text added: "Based on the designs by @Pachuquin & @alvaroalea"
- board text added: "PCB 1.3 by MerlinKV July 27, 2020"
- board text removed: "Original design by @Pachuquin & @alvaroalea"
- board text removed: "PCB MOD 1.3 by MerlinKV July 27, 2020"
Changed lines of the file:
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@@
     (arrow2b (pts (xy 63.5 144.78) (xy 64.626504 144.193579)))
   )
-  (gr_text "PCB MOD 1.3 by MerlinKV\nJuly 27, 2020" (at 142.24 73.66) (layer B.SilkS)
+  (gr_text "PCB 1.3 by MerlinKV\nJuly 27, 2020" (at 142.24 73.66) (layer B.SilkS)
     (effects (font (size 1.5 1.5) (thickness 0.2)) (justify mirror))
   )
@@
   (gr_line (start 86.868 110.49) (end 86.868 124.46) (layer Edge.Cuts) (width 0.15))
   (gr_line (start 63.5 110.49) (end 86.868 110.49) (layer Edge.Cuts) (width 0.15))
-  (gr_text "Original design by\n@Pachuquin & @alvaroalea" (at 87.249 102.616) (layer B.SilkS)
+  (gr_text "Based on the designs by\n@Pachuquin & @alvaroalea" (at 87.249 102.616) (layer B.SilkS)
     (effects (font (size 1.5 1.5) (thickness 0.2)) (justify mirror))
   )
