File: KiCad/PlusD_Clone_1_6.kicad_pcb (KiCad board)
At the start: 2 copper layers, 98.6 x 99.1 mm, 60 parts, among them IC1 WD1772, IC10 74LS27, IC11 GAL22V10, IC2 W27E257, IC3 6224/62256, IC4 GAL20V8B, IC5 74LS06, IC6 74LS126, IC7 74LS374, IC8 74LS175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

Commit message: Add files via upload
Parts:
- IC3: value 6224/62256 -> 6264/62256
Other:
- board text added: "PCB 1.6 by MerlinKV December 1, 2020"
- board text removed: "PCB 1.6 by MerlinKV November 25, 2020"
Changed lines of the file:
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@@
       (effects (font (size 1 1) (thickness 0.15)))
     )
-    (fp_text value 6224/62256 (at 10.721 -2.2686 90) (layer F.SilkS)
+    (fp_text value 6264/62256 (at 10.721 -2.2686 90) (layer F.SilkS)
       (effects (font (size 1 1) (thickness 0.15)))
     )
@@
     (arrow2b (pts (xy 63.5 144.78) (xy 64.626504 144.193579)))
   )
-  (gr_text "PCB 1.6 by MerlinKV\nNovember 25, 2020" (at 142.367 78.232) (layer B.SilkS)
+  (gr_text "PCB 1.6 by MerlinKV\nDecember 1, 2020" (at 142.367 78.232) (layer B.SilkS)
     (effects (font (size 1.5 1.5) (thickness 0.2)) (justify mirror))
   )
