File: KiCad/PlusD_Clone_1_6.sch (KiCad schematic (older format))
At the start: 55 parts, among them IC1 WD1772, IC10 74LS27, IC11 GAL22V10, IC2 W27E257, IC3 6224/62256, IC4 GAL20V8B, IC5 74LS06, IC6 74LS126, IC7 74LS374, IC8 74LS175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

Commit message: Add files via upload
Parts:
- IC3: value 6224/62256 -> 6264/62256
Changed lines of the file:
@@
 Sheet 1 1
 Title "+D Disk Interface Clone"
-Date "2020-10-25"
+Date "2020-12-01"
 Rev "1.6"
 Comp "MerlinKV"
@@
 U 1 1 5F9C4434
 P 6100 1150
-F 0 "IC1" H 6100 1243 39  0000 C CNN
-F 1 "WD1772" H 6100 1168 39  0000 C CNN
+F 0 "IC1" H 6100 1243 47  0000 C CNN
+F 1 "WD1772" H 6100 1168 47  0000 C CNN
 F 2 "Package_DIP:DIP-28_W15.24mm_Socket_LongPads" H 6100 1150 39  0001 C CNN
 F 3 "" H 6100 1150 39  0001 C CNN
@@
 U 1 1 60684FE5
 P 1700 5000
-F 0 "IC4" H 1675 5043 39  0000 C CNN
-F 1 "GAL20V8B" H 1675 4968 39  0000 C CNN
+F 0 "IC4" H 1675 5043 47  0000 C CNN
+F 1 "GAL20V8B" H 1675 4968 47  0000 C CNN
 F 2 "Package_DIP:DIP-24_W7.62mm_Socket_LongPads" H 1700 5000 39  0001 C CNN
 F 3 "" H 1700 5000 39  0001 C CNN
@@
 U 1 1 60991D62
 P 4450 4000
-F 0 "IC3" H 4450 4093 39  0000 C CNN
-F 1 "6224/62256" H 4450 4018 39  0000 C CNN
+F 0 "IC3" H 4450 4093 47  0000 C CNN
+F 1 "6264/62256" H 4450 4018 47  0000 C CNN
 F 2 "Package_DIP:DIP-28_W15.24mm_Socket_LongPads" H 4450 4000 50  0001 C CNN
 F 3 "" H 4450 4000 50  0001 C CNN
@@
 U 1 1 60B20C61
 P 6800 4150
-F 0 "IC8" H 6800 4243 39  0000 C CNN
-F 1 "74LS175" H 6800 4168 39  0000 C CNN
+F 0 "IC8" H 6800 4243 47  0000 C CNN
+F 1 "74LS175" H 6800 4168 47  0000 C CNN
 F 2 "Package_DIP:DIP-16_W7.62mm_Socket_LongPads" H 6800 4150 39  0001 C CNN
 F 3 "" H 6800 4150 39  0001 C CNN
@@
 U 1 1 6103FBDF
 P 9050 6650
-F 0 "IC7" H 9050 6743 39  0000 C CNN
-F 1 "74LS374" H 9050 6668 39  0000 C CNN
+F 0 "IC7" H 9050 6743 47  0000 C CNN
+F 1 "74LS374" H 9050 6668 47  0000 C CNN
 F 2 "Package_DIP:DIP-20_W7.62mm_Socket_LongPads" H 9050 6650 39  0001 C CNN
 F 3 "" H 9050 6650 39  0001 C CNN
